File: Dual-Rail-Power-Supply.kicad_sch (KiCad schematic)
At the start: 0 parts

Commit message: Update schematic and project file with revision details and top-level sheet information
Other:
- title: (none) -> Dual Rail Power Supply
Changed lines of the file:
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@@
 	(generator_version "10.0")
 	(paper "A4")
+	(title_block
+		(title "Dual Rail Power Supply")
+		(date "2026-09-13")
+		(rev "01")
+	)
 	(sheet_instances
 		(path "/"
